File: P1/P1.kicad_pcb (KiCad board)
At the start: 2 copper layers, 64 x 64 mm, 69 parts, among them J1 USB_C, J2 Conn_01x04_Pin, J3 Conn_01x04_Pin, J4 Conn_01x04_Pin, J5 Conn_01x05, J6 Conn_01x05, J7 Conn_01x02_Pin, SW1 SW_SPDT, U1 STM32F103C8T6, U2 MCP2542FD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

Commit message: Reviewed version for manufacture
Parts:
- C1, C2, C3, C6: footprint Capacitor_SMD:C_0402_1005Metric -> Capacitor_SMD:C_0603_1608Metric
- moved C13 2.11 mm to (168.8, 49.6), turned to 90 degrees
- moved C3 0.51 mm to (185.2, 55.2)
- moved C6 0.32 mm to (167.3, 60.4)
Routing:
- net +3.3V: track 263.3 -> 257.3 mm
- net GND: track 51.1 -> 46.1 mm, vias 300 -> 292
Other:
- board text added: "I2C2"

Commit message: Owen Spotted an error, fix
Parts:
- moved C9 1.36 mm to (202.7, 40.4)
Routing:
- net +3.3V: track 257.3 -> 256.6 mm, vias 14 -> 13
- net VBUS: track 57.7 -> 58.2 mm
Changed lines of the file:
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@@
 	(footprint "Capacitor_SMD:C_0603_1608Metric"
 		(layer "F.Cu")
-		(at 201.435 39.9)
+		(at 202.7 40.4)
 		(descr "Capacitor SMD 0603 (1608 Metric), square (rectangular) end terminal, IPC-7351 nominal, (Body size source: IPC-SM-782 page 76, https://www.pcb-3d.com/wordpress/wp-content/uploads/ipc-sm-782a_amendment_1_and_2.pdf), generated with kicad-footprint-generator")
 		(tags "capacitor")
@@
 	)
 	(segment
-		(start 163.41 45.7)
-		(end 163.41 46.24)
-		(width 0.5)
-		(layer "F.Cu")
-		(net 2)
-	)
-	(segment
 		(start 184.35 36.45)
 		(end 184.35 44.6)
@@
 	)
 	(segment
-		(start 163.41 46.24)
-		(end 163.4 46.25)
-		(width 0.5)
-		(layer "F.Cu")
-		(net 2)
-	)
-	(segment
 		(start 169.275 54.275)
 		(end 169.8375 54.8375)
@@
 	)
 	(via
-		(at 163.41 45.7)
-		(size 0.7)
-		(drill 0.3)
-		(layers "F.Cu" "B.Cu")
-		(net 2)
-	)
-	(via
 		(at 167 54)
 		(size 0.7)
@@
 	)
 	(segment
-		(start 163.34 45.77)
-		(end 163.41 45.7)
-		(width 0.5)
-		(layer "B.Cu")
-		(net 2)
-	)
-	(segment
 		(start 166.5 47.7)
 		(end 166.5 50.4)
@@
 	)
 	(segment
-		(start 200.55 40.01)
-		(end 200.66 39.9)
+		(start 183.7 68.85)
+		(end 183.7 66.85)
 		(width 0.5)
 		(layer "F.Cu")
@@
 	)
 	(segment
-		(start 183.7 68.85)
-		(end 183.7 66.85)
+		(start 199.75 40.01)
+		(end 201.535 40.01)
 		(width 0.5)
 		(layer "F.Cu")
@@
 	)
 	(segment
-		(start 198.645 59.32)
-		(end 197.22 59.32)
+		(start 201.535 40.01)
+		(end 201.925 40.4)
 		(width 0.5)
 		(layer "F.Cu")
@@
 	)
 	(segment
-		(start 199.75 40.01)
-		(end 200.55 40.01)
+		(start 198.645 59.32)
+		(end 197.22 59.32)
 		(width 0.5)
 		(layer "F.Cu")
@@
 	)
 	(segment
+		(start 199.75 42.012)
+		(end 201.4 43.662)
+		(width 0.5)
+		(layer "B.Cu")
+		(net 7)
+	)
+	(segment
 		(start 200.5 57.6)
 		(end 200.5 56.1)
@@
 	)
 	(segment
+		(start 199.75 40.01)
+		(end 199.75 42.012)
+		(width 0.5)
+		(layer "B.Cu")
+		(net 7)
+	)
+	(segment
 		(start 196.4 54.5)
 		(end 198 56.1)
@@
 		(width 0.5)
 		(layer "B.Cu")
-		(net 7)
-	)
-	(segment
-		(start 201.4 43.662)
-		(end 198.749 41.011)
-		(width 0.5)
-		(layer "B.Cu")
-		(net 7)
-	)
-	(segment
-		(start 198.749 41.011)
-		(end 199.75 40.01)
-		(width 0.5)
-		(layer "B.Cu")
